File: src/ESP32-Sensor-PCB.kicad_pcb (KiCad board)
At the start: 2 copper layers, 28 x 28 mm, 3 parts, among them U1 XIAO-ESP32-S3-SMD, U2 HDC1080DMBR

Commit message: v1.1
Other:
- board text added: "XIAO HERE"
- board text added: "sensor ->"
Changed lines of the file:
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@@
 			(at 0 0.254 0)
 			(layer "F.SilkS")
+			(hide yes)
 			(effects
 				(font
@@
 			(at -7.747 -7.62 0)
 			(layer "F.Fab")
+			(hide yes)
 			(effects
 				(font
@@
 		)
 	)
+	(gr_text "XIAO HERE"
+		(at 85 64.5 0)
+		(layer "B.SilkS")
+		(effects
+			(font
+				(size 1.5 1.5)
+				(thickness 0.3)
+				(bold yes)
+			)
+			(justify left bottom mirror)
+		)
+	)
+	(gr_text "sensor ->"
+		(at 65.5 68.5 270)
+		(layer "B.SilkS")
+		(effects
+			(font
+				(size 1 1)
+				(thickness 0.2)
+				(bold yes)
+			)
+			(justify left bottom mirror)
+		)
+	)
